File: I2C-7-Segment-Backpack-dot8inch.brd (EAGLE design)
At the start: 45.7 x 40.6 mm, 21 parts, among them J1 4P-SMD-2.0-90D, J2 4P-SMD-2.0-90D, U1 AS1115

Commit message: Rev C
Other:
- board text added: "0.8 inch LED - (Rev C)"
- board text added: "I2C 7 SEGMENT BKPK .8" (Rev C)"
- board text added: "dcity.org"
- board text removed: "0.8 inch LED - (Rev B)"
- board text removed: "I2C 7 SEGMENT BKPK .8" (Rev B)"
- board text removed: "wht.io"
Changed lines of the file:
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@@
 <?xml version="1.0" encoding="utf-8"?>
 <!DOCTYPE eagle SYSTEM "eagle.dtd">
-<eagle version="7.5.0">
+<eagle version="9.1.3">
 <drawing>
 <settings>
 <setting alwaysvectorfont="no"/>
+<setting keepoldvectorfont="yes"/>
 <setting verticaltext="up"/>
 </settings>
@@
 <text x="28.829" y="13.081" size="0.889" layer="21" font="vector" ratio="15" rot="R180">GND</text>
 <text x="12.192" y="3.81" size="0.889" layer="21" font="vector" ratio="15">I2C - 7 Segment Backpack</text>
-<text x="12.319" y="2.54" size="0.889" layer="21" font="vector" ratio="15">0.8 inch LED -  (Rev B)</text>
+<text x="12.319" y="2.54" size="0.889" layer="21" font="vector" ratio="15">0.8 inch LED -  (Rev C)</text>
 <text x="7.62" y="38.1" size="0.889" layer="21" font="vector" ratio="15">SET I2C ADDR WITH SJ3 AND SJ4</text>
 <text x="7.62" y="35.56" size="0.889" layer="21" font="vector" ratio="15">BOTH OPEN = 03h</text>
@@
 <text x="7.62" y="36.83" size="0.889" layer="21" font="vector" ratio="15">SJ3 CLOSED = 01h</text>
 <text x="24.13" y="35.56" size="0.889" layer="21" font="vector" ratio="15">DO NOT CLOSE BOTH</text>
-<text x="33.02" y="3.81" size="0.889" layer="22" font="vector" ratio="15" rot="MR0">I2C 7 SEGMENT BKPK .8" (Rev B)</text>
+<text x="33.02" y="3.81" size="0.889" layer="22" font="vector" ratio="15" rot="MR0">I2C 7 SEGMENT BKPK .8" (Rev C)</text>
 <text x="30.607" y="7.62" size="0.889" layer="21" font="vector" ratio="15" rot="R180">LED1</text>
 <text x="28.067" y="6.985" size="0.889" layer="22" font="vector" ratio="15" rot="MR180">LED1</text>
@@
 <rectangle x1="29.464" y1="22.352" x2="31.242" y2="23.749" layer="43"/>
 <rectangle x1="17.78" y1="26.924" x2="19.558" y2="28.194" layer="43"/>
-<text x="32.131" y="1.143" size="1.524" layer="21" font="vector" ratio="10">wht.io</text>
-<text x="38.1" y="1.27" size="1.524" layer="22" font="vector" ratio="10" rot="MR0">wht.io</text>
+<text x="27.051" y="1.143" size="1.524" layer="21" font="vector" ratio="10">dcity.org</text>
+<text x="38.1" y="1.27" size="1.524" layer="22" font="vector" ratio="10" rot="MR0">dcity.org</text>
 </plain>
 <attributes>
@@
 <param name="dpMaxLengthDifference" value="10mm"/>
 <param name="dpGapFactor" value="2.5"/>
-<param name="checkGrid" value="0"/>
 <param name="checkAngle" value="1"/>
 <param name="checkFont" value="1"/>
 <param name="checkRestrict" value="1"/>
+<param name="checkStop" value="0"/>
+<param name="checkValues" value="0"/>
+<param name="checkNames" value="1"/>
+<param name="checkWireStubs" value="1"/>
+<param name="checkPolygonWidth" value="0"/>
 <param name="useDiameter" value="13"/>
 <param name="maxErrors" value="50"/>
@@
 </signal>
 </signals>
+<mfgpreviewcolors>
+<mfgpreviewcolor name="soldermaskcolor" color="0xC8008000"/>
+<mfgpreviewcolor name="silkscreencolor" color="0xFFFEFEFE"/>
+<mfgpreviewcolor name="backgroundcolor" color="0xFF282828"/>
+<mfgpreviewcolor name="coppercolor" color="0xFFFFBF00"/>
+<mfgpreviewcolor name="substratecolor" color="0xFF786E46"/>
+</mfgpreviewcolors>
 </board>
 </drawing>

Commit message: Rev D
Parts:
- J1, J2: value 4P-SMD-2.0-90D -> QWIIC_RIGHT_ANGLE; device 0:HW4-SMD-2.0-90D -> 0:JST04_1MM_RA
- moved J1 30.5 mm to (5.08, 16.5)
- moved J2 29.2 mm to (40.6, 16.5)
Connections:
- net GND: now also J1.1, J2.1; no longer J1.4, J2.4
- net SCL: now also J1.4, J2.4; no longer J1.1, J2.1
- net SDA: now also J1.3, J2.3; no longer J1.2, J2.2
- net VCC: now also J1.2, J2.2; no longer J1.3, J2.3
Routing:
- net SCL: track 66.1 -> 96.9 mm
- net SDA: track 70.6 -> 81.5 mm
- net VCC: track 112.0 -> 120.2 mm
- net N$5: track 28.5 -> 34.7 mm
- net GND: track 17.2 -> 11.1 mm
- net N$11: track 13.3 -> 10.2 mm
- net N$14: track 37.0 -> 38.2 mm
Other:
- board text added: "0.8 inch LED - (Rev D)"
- board text added: "I2C 7 SEGMENT BKPK .8" (Rev D)"
- board text removed: "0.8 inch LED - (Rev C)"
- board text removed: "I2C 7 SEGMENT BKPK .8" (Rev C)"
