File: I2C-7-Segment-Backpack-dot8inch.sch (EAGLE design)
At the start: 21 parts, among them J1 4P-SMD-2.0-90D, J2 4P-SMD-2.0-90D, U1 AS1115

Commit message: Rev D
Parts:
- J1, J2: value 4P-SMD-2.0-90D -> QWIIC_RIGHT_ANGLE; device 0:GROVE-CONNECTOR-SMD-90D(4+2P-2.0) -> 0:QWIIC_CONNECTORJS-1MM
Connections:
- net GND: now also J1.1, J2.1; no longer J1.4, J2.4
- net SCL: now also J1.4, J2.4; no longer J1.1, J2.1
- net SDA: now also J1.3, J2.3; no longer J1.2, J2.2
- net VCC: now also J1.2, J2.2; no longer J1.3, J2.3
Other:
- moved on the sheet: J3
